Commit message: This is now a ROS2 package. Added also ros2_control and an imu sensor on the base.

File: urdf/anymal.xacro (robot description, xacro)
@@ -4,5 +4,11 @@
 <!-- =================================================================================== -->
 <!-- This file contains the description of the ANYmal C robot. -->
-<robot name="anymal">
+<robot name="anymal" xmlns:xacro="http://www.ros.org/wiki/xacro">
+    <!-- Constants for robot dimensions -->
+    <xacro:property name="PI" value="3.1415926535897931"/>
+    <!-- Import all Gazebo-customization elements, including Gazebo colors -->
+    <xacro:include filename="$(find anymal_c_simple_description)/urdf/anymal_gazebo.xacro" />
+    <!-- Import Rviz colors -->
+    <xacro:include filename="$(find anymal_c_simple_description)/urdf/materials.xacro" />
     <!-- Base link -->
     <link name="base">

Commit message: Removed shanks collisions

File: urdf/anymal.xacro (robot description, xacro)
@@ -832,10 +832,10 @@
         </visual>
         <!-- Adapter collision -->
-        <collision>
+        <!-- <collision>
             <origin rpy="0 0 0" xyz="0 0 0.168985"/>
             <geometry>
                 <cylinder length="0.282504" radius="0.0175"/>
             </geometry>
-        </collision>
+        </collision> -->
         <!-- Foot collision -->
         <collision>
@@ -1076,10 +1076,10 @@
         </visual>
         <!-- Adapter collision -->
-        <collision>
+        <!-- <collision>
             <origin rpy="0 0 0" xyz="0 0 0.168985"/>
             <geometry>
                 <cylinder length="0.282504" radius="0.0175"/>
             </geometry>
-        </collision>
+        </collision> -->
         <!-- Foot collision -->
         <collision>
@@ -1320,10 +1320,10 @@
         </visual>
         <!-- Adapter collision -->
-        <collision>
+        <!-- <collision>
             <origin rpy="0 0 0" xyz="0 0 0.168985"/>
             <geometry>
                 <cylinder length="0.282504" radius="0.0175"/>
             </geometry>
-        </collision>
+        </collision> -->
         <!-- Foot collision -->
         <collision>
@@ -1564,10 +1564,10 @@
         </visual>
         <!-- Adapter collision -->
-        <collision>
+        <!-- <collision>
             <origin rpy="0 0 0" xyz="0 0 0.168985"/>
             <geometry>
                 <cylinder length="0.282504" radius="0.0175"/>
             </geometry>
-        </collision>
+        </collision> -->
         <!-- Foot collision -->
         <collision>

File: urdf/anymal_gazebo.xacro (robot description, xacro)
@@ -125,5 +125,5 @@
             <contact>
                 <!-- gz sdf -p turtlebot3_burger.urdf.xacro and look for the name of the desired collision element. -->
-                <collision>LF_SHANK_fixed_joint_lump__LF_FOOT_collision_3</collision>
+                <collision>LF_SHANK_fixed_joint_lump__LF_FOOT_collision_2</collision>
             </contact>
             <plugin name="LF_FOOT_bumper" filename="libgazebo_ros_bumper.so">
@@ -143,5 +143,5 @@
             <contact>
                 <!-- gz sdf -p turtlebot3_burger.urdf.xacro and look for the name of the desired collision element. -->
-                <collision>RF_SHANK_fixed_joint_lump__RF_FOOT_collision_3</collision>
+                <collision>RF_SHANK_fixed_joint_lump__RF_FOOT_collision_2</collision>
             </contact>
             <plugin name="RF_FOOT_bumper" filename="libgazebo_ros_bumper.so">
@@ -161,5 +161,5 @@
             <contact>
                 <!-- gz sdf -p turtlebot3_burger.urdf.xacro and look for the name of the desired collision element. -->
-                <collision>LH_SHANK_fixed_joint_lump__LH_FOOT_collision_3</collision>
+                <collision>LH_SHANK_fixed_joint_lump__LH_FOOT_collision_2</collision>
             </contact>
             <plugin name="LH_FOOT_bumper" filename="libgazebo_ros_bumper.so">
@@ -179,5 +179,5 @@
             <contact>
                 <!-- gz sdf -p turtlebot3_burger.urdf.xacro and look for the name of the desired collision element. -->
-                <collision>RH_SHANK_fixed_joint_lump__RH_FOOT_collision_3</collision>
+                <collision>RH_SHANK_fixed_joint_lump__RH_FOOT_collision_2</collision>
             </contact>
             <plugin name="RH_FOOT_bumper" filename="libgazebo_ros_bumper.so">

Commit message: Added a xacro arg to avoid loading the gazebo part

File: urdf/anymal.xacro (robot description, xacro)
@@ -5,10 +5,14 @@
 <!-- This file contains the description of the ANYmal C robot. -->
 <robot name="anymal" xmlns:xacro="http://www.ros.org/wiki/xacro">
+    <xacro:arg name="use_gazebo" default="True"/>
+    <xacro:property name="use_gazebo" default="$(arg use_gazebo)"/>
     <!-- Constants for robot dimensions -->
     <xacro:property name="PI" value="3.1415926535897931"/>
     <!-- Import all Gazebo-customization elements, including Gazebo colors -->
-    <xacro:include filename="$(find anymal_c_simple_description)/urdf/anymal_gazebo.xacro" />
+    <xacro:if value="${use_gazebo}">
+        <xacro:include filename="$(find anymal_c_simple_description)/urdf/anymal_gazebo.xacro"/>
+    </xacro:if>
     <!-- Import Rviz colors -->
-    <xacro:include filename="$(find anymal_c_simple_description)/urdf/materials.xacro" />
+    <xacro:include filename="$(find anymal_c_simple_description)/urdf/materials.xacro"/>
     <gazebo>
         <static>false</static>

Commit message: Added xacro arg to remove shank collisions

File: urdf/anymal.xacro (robot description, xacro)
@@ -7,4 +7,6 @@
     <xacro:arg name="use_gazebo" default="True"/>
     <xacro:property name="use_gazebo" default="$(arg use_gazebo)"/>
+    <xacro:arg name="remove_collisions" default="False"/>
+    <xacro:property name="remove_collisions" default="$(arg remove_collisions)"/>
     <!-- Constants for robot dimensions -->
     <xacro:property name="PI" value="3.1415926535897931"/>
@@ -839,10 +841,12 @@
         </visual>
         <!-- Adapter collision -->
-        <!-- <collision>
-            <origin rpy="0 0 0" xyz="0 0 0.168985"/>
-            <geometry>
-                <cylinder length="0.282504" radius="0.0175"/>
-            </geometry>
-        </collision> -->
+        <xacro:unless value="${remove_collisions}">
+            <collision>
+                <origin rpy="0 0 0" xyz="0 0 0.168985"/>
+                <geometry>
+                    <cylinder length="0.282504" radius="0.0175"/>
+                </geometry>
+            </collision>
+        </xacro:unless>
         <!-- Foot collision -->
         <collision>
@@ -1083,10 +1087,12 @@
         </visual>
         <!-- Adapter collision -->
-        <!-- <collision>
-            <origin rpy="0 0 0" xyz="0 0 0.168985"/>
-            <geometry>
-                <cylinder length="0.282504" radius="0.0175"/>
-            </geometry>
-        </collision> -->
+        <xacro:unless value="${remove_collisions}">
+            <collision>
+                <origin rpy="0 0 0" xyz="0 0 0.168985"/>
+                <geometry>
+                    <cylinder length="0.282504" radius="0.0175"/>
+                </geometry>
+            </collision>
+        </xacro:unless>
         <!-- Foot collision -->
         <collision>
@@ -1327,10 +1333,12 @@
         </visual>
         <!-- Adapter collision -->
-        <!-- <collision>
-            <origin rpy="0 0 0" xyz="0 0 0.168985"/>
-            <geometry>
-                <cylinder length="0.282504" radius="0.0175"/>
-            </geometry>
-        </collision> -->
+        <xacro:unless value="${remove_collisions}">
+            <collision>
+                <origin rpy="0 0 0" xyz="0 0 0.168985"/>
+                <geometry>
+                    <cylinder length="0.282504" radius="0.0175"/>
+                </geometry>
+            </collision>
+        </xacro:unless>
         <!-- Foot collision -->
         <collision>
@@ -1571,10 +1579,12 @@
         </visual>
         <!-- Adapter collision -->
-        <!-- <collision>
-            <origin rpy="0 0 0" xyz="0 0 0.168985"/>
-            <geometry>
-                <cylinder length="0.282504" radius="0.0175"/>
-            </geometry>
-        </collision> -->
+        <xacro:unless value="${remove_collisions}">
+            <collision>
+                <origin rpy="0 0 0" xyz="0 0 0.168985"/>
+                <geometry>
+                    <cylinder length="0.282504" radius="0.0175"/>
+                </geometry>
+            </collision>
+        </xacro:unless>
         <!-- Foot collision -->
         <collision>

Commit message: Contact sensor bug fix

File: urdf/anymal.xacro (robot description, xacro)
@@ -7,6 +7,6 @@
     <xacro:arg name="use_gazebo" default="True"/>
     <xacro:property name="use_gazebo" default="$(arg use_gazebo)"/>
-    <xacro:arg name="remove_collisions" default="False"/>
-    <xacro:property name="remove_collisions" default="$(arg remove_collisions)"/>
+    <xacro:arg name="remove_shank_collisions" default="False"/>
+    <xacro:property name="remove_shank_collisions" default="$(arg remove_shank_collisions)"/>
     <!-- Constants for robot dimensions -->
     <xacro:property name="PI" value="3.1415926535897931"/>
@@ -841,5 +841,5 @@
         </visual>
         <!-- Adapter collision -->
-        <xacro:unless value="${remove_collisions}">
+        <xacro:unless value="${remove_shank_collisions}">
             <collision>
                 <origin rpy="0 0 0" xyz="0 0 0.168985"/>
@@ -1087,5 +1087,5 @@
         </visual>
         <!-- Adapter collision -->
-        <xacro:unless value="${remove_collisions}">
+        <xacro:unless value="${remove_shank_collisions}">
             <collision>
                 <origin rpy="0 0 0" xyz="0 0 0.168985"/>
@@ -1333,5 +1333,5 @@
         </visual>
         <!-- Adapter collision -->
-        <xacro:unless value="${remove_collisions}">
+        <xacro:unless value="${remove_shank_collisions}">
             <collision>
                 <origin rpy="0 0 0" xyz="0 0 0.168985"/>
@@ -1579,5 +1579,5 @@
         </visual>
         <!-- Adapter collision -->
-        <xacro:unless value="${remove_collisions}">
+        <xacro:unless value="${remove_shank_collisions}">
             <collision>
                 <origin rpy="0 0 0" xyz="0 0 0.168985"/>

File: urdf/anymal_gazebo.xacro (robot description, xacro)
@@ -125,5 +125,10 @@
             <contact>
                 <!-- gz sdf -p turtlebot3_burger.urdf.xacro and look for the name of the desired collision element. -->
-                <collision>LF_SHANK_fixed_joint_lump__LF_FOOT_collision_2</collision>
+                <xacro:if value="${remove_shank_collisions}">
+                    <collision>LF_SHANK_fixed_joint_lump__LF_FOOT_collision_2</collision>
+                </xacro:if>
+                <xacro:unless value="${remove_shank_collisions}">
+                    <collision>LF_SHANK_fixed_joint_lump__LF_FOOT_collision_3</collision>
+                </xacro:unless>
             </contact>
             <plugin name="LF_FOOT_bumper" filename="libgazebo_ros_bumper.so">
@@ -143,5 +148,10 @@
             <contact>
                 <!-- gz sdf -p turtlebot3_burger.urdf.xacro and look for the name of the desired collision element. -->
-                <collision>RF_SHANK_fixed_joint_lump__RF_FOOT_collision_2</collision>
+                <xacro:if value="${remove_shank_collisions}">
+                    <collision>RF_SHANK_fixed_joint_lump__RF_FOOT_collision_2</collision>
+                </xacro:if>
+                <xacro:unless value="${remove_shank_collisions}">
+                    <collision>RF_SHANK_fixed_joint_lump__RF_FOOT_collision_3</collision>
+                </xacro:unless>
             </contact>
             <plugin name="RF_FOOT_bumper" filename="libgazebo_ros_bumper.so">
@@ -161,5 +171,10 @@
             <contact>
                 <!-- gz sdf -p turtlebot3_burger.urdf.xacro and look for the name of the desired collision element. -->
-                <collision>LH_SHANK_fixed_joint_lump__LH_FOOT_collision_2</collision>
+                <xacro:if value="${remove_shank_collisions}">
+                    <collision>LH_SHANK_fixed_joint_lump__LH_FOOT_collision_2</collision>
+                </xacro:if>
+                <xacro:unless value="${remove_shank_collisions}">
+                    <collision>LH_SHANK_fixed_joint_lump__LH_FOOT_collision_3</collision>
+                </xacro:unless>
             </contact>
             <plugin name="LH_FOOT_bumper" filename="libgazebo_ros_bumper.so">
@@ -179,5 +194,10 @@
             <contact>
                 <!-- gz sdf -p turtlebot3_burger.urdf.xacro and look for the name of the desired collision element. -->
-                <collision>RH_SHANK_fixed_joint_lump__RH_FOOT_collision_2</collision>
+                <xacro:if value="${remove_shank_collisions}">
+                    <collision>RH_SHANK_fixed_joint_lump__RH_FOOT_collision_2</collision>
+                </xacro:if>
+                <xacro:unless value="${remove_shank_collisions}">
+                    <collision>RH_SHANK_fixed_joint_lump__RH_FOOT_collision_3</collision>
+                </xacro:unless>
             </contact>
             <plugin name="RH_FOOT_bumper" filename="libgazebo_ros_bumper.so">

Commit message: Add argument to fix base in place (for debugging)

File: urdf/anymal.xacro (robot description, xacro)
@@ -9,5 +9,7 @@
     <xacro:arg name="remove_shank_collisions" default="False"/>
     <xacro:property name="remove_shank_collisions" default="$(arg remove_shank_collisions)"/>
-    <!-- Constants for robot dimensions -->
+    <xacro:arg name="static" default="False"/>
+    <xacro:arg name="use_gazebo" default="True"/>
+    <xacro:property name="use_gazebo" default="$(arg use_gazebo)"/>
     <xacro:property name="PI" value="3.1415926535897931"/>
     <!-- Import all Gazebo-customization elements, including Gazebo colors -->
@@ -17,7 +19,9 @@
     <!-- Import Rviz colors -->
     <xacro:include filename="$(find anymal_c_simple_description)/urdf/materials.xacro"/>
-    <gazebo>
-        <static>false</static>
+    <xacro:if value="$(arg debug)">
+    <gazebo reference="base">
+        <kinematic>false</kinematic>
     </gazebo>
+    </xacro:if>
     <!-- Base link -->
     <link name="base">
