Commit message: Remove all comments

File: urdf/anymal.xacro (robot description, xacro)
@@ -1,10 +1,4 @@
 <?xml version="1.0" encoding="utf-8"?>
-<!-- =================================================================================== -->
-<!--   Copyright 2020 ANYbotics, https://www.anybotics.com                               -->
-<!-- =================================================================================== -->
-<!-- This file contains the description of the ANYmal C robot. -->
 <robot name="anymal" xmlns:xacro="http://www.ros.org/wiki/xacro">
-    <xacro:arg name="use_gazebo" default="True"/>
-    <xacro:property name="use_gazebo" default="$(arg use_gazebo)"/>
     <xacro:arg name="remove_shank_collisions" default="False"/>
     <xacro:property name="remove_shank_collisions" default="$(arg remove_shank_collisions)"/>
@@ -13,16 +7,13 @@
     <xacro:property name="use_gazebo" default="$(arg use_gazebo)"/>
     <xacro:property name="PI" value="3.1415926535897931"/>
-    <!-- Import all Gazebo-customization elements, including Gazebo colors -->
     <xacro:if value="${use_gazebo}">
         <xacro:include filename="$(find anymal_c_simple_description)/urdf/anymal_gazebo.xacro"/>
     </xacro:if>
-    <!-- Import Rviz colors -->
     <xacro:include filename="$(find anymal_c_simple_description)/urdf/materials.xacro"/>
     <xacro:if value="$(arg debug)">
-    <gazebo reference="base">
-        <kinematic>false</kinematic>
-    </gazebo>
+        <gazebo reference="base">
+            <kinematic>false</kinematic>
+        </gazebo>
     </xacro:if>
-    <!-- Base link -->
     <link name="base">
         <visual>
@@ -62,5 +53,4 @@
             </geometry>
         </collision>
-        <!-- Shell self filtering -->
         <self_filter>
             <origin rpy="0 0 0" xyz="0 0 0"/>
@@ -70,5 +60,4 @@
         </self_filter>
     </link>
-    <!-- Fixed joint to add dummy inertia link -->
     <joint name="base_to_base_inertia" type="fixed">
         <parent link="base"/>
@@ -76,5 +65,4 @@
         <origin rpy="0 0 0" xyz="0 0 0"/>
     </joint>
-    <!-- Dummy inertia link, because KDL cannot have inertia on the base link -->
     <link name="base_inertia">
         <inertial>
@@ -84,5 +72,4 @@
         </inertial>
     </link>
-    <!-- Fixed joint base topshell -->
     <joint name="base_top_shell" type="fixed">
         <parent link="base"/>
@@ -90,5 +77,4 @@
         <origin rpy="0 0 0" xyz="0 0 0"/>
     </joint>
-    <!-- Top shell link -->
     <link name="top_shell">
         <visual>
@@ -104,5 +90,4 @@
         </inertial>
     </link>
-    <!-- Fixed joint base topshell -->
     <joint name="base_bottom_shell" type="fixed">
         <parent link="base"/>
@@ -110,5 +95,4 @@
         <origin rpy="0 0 0" xyz="0 0 0"/>
     </joint>
-    <!-- Bottom shell link -->
     <link name="bottom_shell">
         <visual>
@@ -124,5 +108,4 @@
         </inertial>
     </link>
-    <!-- Fixed joint base remote -->
     <joint name="base_remote" type="fixed">
         <parent link="base"/>
@@ -130,5 +113,4 @@
         <origin rpy="0 0 0" xyz="0 0 0"/>
     </joint>
-    <!-- Remote link -->
     <link name="remote">
         <visual>
@@ -144,5 +126,4 @@
         </inertial>
     </link>
-    <!-- Fixed joint base handle -->
     <joint name="base_handle" type="fixed">
         <parent link="base"/>
@@ -150,5 +131,4 @@
         <origin rpy="0 0 0" xyz="0 0 0"/>
     </joint>
-    <!-- Handle link -->
     <link name="handle">
         <visual>
@@ -164,5 +144,4 @@
         </inertial>
     </link>
-    <!-- Fixed joint base face -->
     <joint name="base_face_front" type="fixed">
         <parent link="base"/>
@@ -170,5 +149,4 @@
         <origin rpy="0 0 -0.0" xyz="0.4145 0 0"/>
     </joint>
-    <!-- Shell link -->
     <link name="face_front">
         <visual>
@@ -202,6 +180,4 @@
         </inertial>
     </link>
-    <!-- Camera joint -->
-    <!-- Is located between the two back screw holes at ground level. -->
     <joint name="face_front_to_depth_camera_front_camera" type="fixed">
         <parent link="face_front"/>
@@ -209,5 +185,4 @@
         <origin rpy="0.0 0.523598775598 0" xyz="0.04715 0.0 -0.0292"/>
     </joint>
-    <!-- Camera link -->
     <link name="depth_camera_front_camera">
         <visual>
@@ -223,6 +198,4 @@
         </inertial>
     </link>
-    <!-- Camera parent joint -->
-    <!-- Frame lies on the left ir camera according to any_realsense2_camera urdf. -->
     <joint name="depth_camera_front_camera_to_camera_parent" type="fixed">
         <parent link="depth_camera_front_camera"/>
@@ -230,7 +203,5 @@
         <origin rpy="0.0 0.0 0.0" xyz="0.0255 0.0175 0.0"/>
     </joint>
-    <!-- Camera parent link -->
     <link name="depth_camera_front_camera_parent"/>
-    <!-- Depth optical frame joint -->
     <joint name="depth_camera_front_camera_parent_to_depth_optical_frame" type="fixed">
         <parent link="depth_camera_front_camera_parent"/>
@@ -238,7 +209,5 @@
         <origin rpy="-1.57079632679 0.0 -1.57079632679" xyz="0.0 0.0 0.0"/>
     </joint>
-    <!-- Depth optical frame link -->
     <link name="depth_camera_front_depth_optical_frame"/>
-    <!-- Camera color frame joint -->
     <joint name="depth_camera_front_camera_parent_to_color_frame" type="fixed">
         <parent link="depth_camera_front_camera_parent"/>
@@ -246,7 +215,5 @@
         <origin rpy="0 0 0" xyz="0 0.015 0"/>
     </joint>
-    <!-- Camera color frame link -->
     <link name="depth_camera_front_color_frame"/>
-    <!-- Camera color optical joint -->
     <joint name="depth_camera_front_color_frame_to_color_optical_frame" type="fixed">
         <parent link="depth_camera_front_color_frame"/>
@@ -254,8 +221,5 @@
         <origin rpy="-1.57079632679 0.0 -1.57079632679" xyz="0.0 0.0 0.0"/>
     </joint>
-    <!-- Camera color optical link -->
     <link name="depth_camera_front_color_optical_frame"/>
-    <!-- Camera joint -->
-    <!-- Is located in the center of the mounting points. -->
     <joint name="face_front_to_wide_angle_camera_front_camera" type="fixed">
         <parent link="face_front"/>
@@ -263,5 +227,4 @@
         <origin rpy="0 0 0" xyz="0.09850 0.0 0.01497"/>
     </joint>
-    <!-- Camera link -->
     <link name="wide_angle_camera_front_camera">
         <visual>
@@ -277,5 +240,4 @@
         </inertial>
     </link>
-    <!-- Camera parent joint -->
     <joint name="wide_angle_camera_front_camera_to_camera_parent" type="fixed">
         <parent link="wide_angle_camera_front_camera"/>
@@ -283,7 +245,5 @@
         <origin rpy="-1.57079632679 0.0 -1.57079632679" xyz="0.0 0.0 0.0"/>
     </joint>
-    <!-- Camera parent link -->
     <link name="wide_angle_camera_front_camera_parent"/>
-    <!-- Fixed joint base face -->
     <joint name="base_face_rear" type="fixed">
         <parent link="base"/>
@@ -291,5 +251,4 @@
         <origin rpy="0 0 3.14159265359" xyz="-0.4145 0 0"/>
     </joint>
-    <!-- Shell link -->
     <link name="face_rear">
         <visual>
@@ -323,6 +282,4 @@
         </inertial>
     </link>
-    <!-- Camera joint -->
-    <!-- Is located between the two back screw holes at ground level. -->
     <joint name="face_rear_to_depth_camera_rear_camera" type="fixed">
         <parent link="face_rear"/>
@@ -330,5 +287,4 @@
         <origin rpy="0.0 0.523598775598 0" xyz="0.04715 0.0 -0.0292"/>
     </joint>
-    <!-- Camera link -->
     <link name="depth_camera_rear_camera">
         <visual>
@@ -344,6 +300,4 @@
         </inertial>
     </link>
-    <!-- Camera parent joint -->
-    <!-- Frame lies on the left ir camera according to any_realsense2_camera urdf. -->
     <joint name="depth_camera_rear_camera_to_camera_parent" type="fixed">
         <parent link="depth_camera_rear_camera"/>
@@ -351,7 +305,5 @@
         <origin rpy="0.0 0.0 0.0" xyz="0.0255 0.0175 0.0"/>
     </joint>
-    <!-- Camera parent link -->
     <link name="depth_camera_rear_camera_parent"/>
-    <!-- Depth optical frame joint -->
     <joint name="depth_camera_rear_camera_parent_to_depth_optical_frame" type="fixed">
         <parent link="depth_camera_rear_camera_parent"/>
@@ -359,7 +311,5 @@
         <origin rpy="-1.57079632679 0.0 -1.57079632679" xyz="0.0 0.0 0.0"/>
     </joint>
-    <!-- Depth optical frame link -->
     <link name="depth_camera_rear_depth_optical_frame"/>
-    <!-- Camera color frame joint -->
     <joint name="depth_camera_rear_camera_parent_to_color_frame" type="fixed">
         <parent link="depth_camera_rear_camera_parent"/>
@@ -367,7 +317,5 @@
         <origin rpy="0 0 0" xyz="0 0.015 0"/>
     </joint>
-    <!-- Camera color frame link -->
     <link name="depth_camera_rear_color_frame"/>
-    <!-- Camera color optical joint -->
     <joint name="depth_camera_rear_color_frame_to_color_optical_frame" type="fixed">
         <parent link="depth_camera_rear_color_frame"/>
@@ -375,8 +323,5 @@
         <origin rpy="-1.57079632679 0.0 -1.57079632679" xyz="0.0 0.0 0.0"/>
     </joint>
-    <!-- Camera color optical link -->
     <link name="depth_camera_rear_color_optical_frame"/>
-    <!-- Camera joint -->
-    <!-- Is located in the center of the mounting points. -->
     <joint name="face_rear_to_wide_angle_camera_rear_camera" type="fixed">
         <parent link="face_rear"/>
@@ -384,5 +329,4 @@
         <origin rpy="0 0 0" xyz="0.09850 0.0 0.01497"/>
     </joint>
-    <!-- Camera link -->
     <link name="wide_angle_camera_rear_camera">
         <visual>
@@ -398,5 +342,4 @@
         </inertial>
     </link>
-    <!-- Camera parent joint -->
     <joint name="wide_angle_camera_rear_camera_to_camera_parent" type="fixed">
         <parent link="wide_angle_camera_rear_camera"/>
@@ -404,7 +347,5 @@
         <origin rpy="-1.57079632679 0.0 -1.57079632679" xyz="0.0 0.0 0.0"/>
     </joint>
-    <!-- Camera parent link -->
     <link name="wide_angle_camera_rear_camera_parent"/>
-    <!-- Fixed joint base battery -->
     <joint name="base_battery" type="fixed">
         <parent link="base"/>
@@ -412,5 +353,4 @@
         <origin rpy="0 0 0" xyz="0 0 0"/>
     </joint>
-    <!-- Shell link -->
     <link name="battery">
         <visual>
@@ -426,5 +366,4 @@
         </inertial>
     </link>
-    <!-- Fixed joint to add docking  -->
     <joint name="base_to_docking_hatch_cover" type="fixed">
         <parent link="base"/>
@@ -432,7 +371,5 @@
         <origin rpy="0 0 0" xyz="0.343 0.0 -0.07"/>
     </joint>
-    <!-- Hatch cover link -->
     <link name="docking_hatch_cover">
-        <!--  TODO(fgiraldez): add visual    -->
         <inertial>
             <origin rpy="0 0 0" xyz="-0.003 0.0 0.005"/>
@@ -447,5 +384,4 @@
                 <box size="0.024 0.024 0.01"/>
             </geometry>
-            <!-- <material name="orange"/> -->
         </visual>
         <collision>
@@ -466,6 +402,4 @@
         <origin rpy="0.0 0.0 1.57079632679" xyz="0.2488 0.00835 0.04628"/>
     </joint>
-    <!-- Camera joint -->
-    <!-- Is located between the two back screw holes at ground level. -->
     <joint name="base_to_depth_camera_left_camera" type="fixed">
         <parent link="base"/>
@@ -473,5 +407,4 @@
         <origin rpy="0.0 0.523598775598 1.57079632679" xyz="0.0 0.07646 0.02905"/>
     </joint>
-    <!-- Camera link -->
     <link name="depth_camera_left_camera">
         <visual>
@@ -487,6 +420,4 @@
         </inertial>
     </link>
-    <!-- Camera parent joint -->
-    <!-- Frame lies on the left ir camera according to any_realsense2_camera urdf. -->
     <joint name="depth_camera_left_camera_to_camera_parent" type="fixed">
         <parent link="depth_camera_left_camera"/>
@@ -494,7 +425,5 @@
         <origin rpy="0.0 0.0 0.0" xyz="0.0255 0.0175 0.0"/>
     </joint>
-    <!-- Camera parent link -->
     <link name="depth_camera_left_camera_parent"/>
-    <!-- Depth optical frame joint -->
     <joint name="depth_camera_left_camera_parent_to_depth_optical_frame" type="fixed">
         <parent link="depth_camera_left_camera_parent"/>
@@ -502,7 +431,5 @@
         <origin rpy="-1.57079632679 0.0 -1.57079632679" xyz="0.0 0.0 0.0"/>
     </joint>
-    <!-- Depth optical frame link -->
     <link name="depth_camera_left_depth_optical_frame"/>
-    <!-- Camera color frame joint -->
     <joint name="depth_camera_left_camera_parent_to_color_frame" type="fixed">
         <parent link="depth_camera_left_camera_parent"/>
@@ -510,7 +437,5 @@
         <origin rpy="0 0 0" xyz="0 0.015 0"/>
     </joint>
-    <!-- Camera color frame link -->
     <link name="depth_camera_left_color_frame"/>
-    <!-- Camera color optical joint -->
     <joint name="depth_camera_left_color_frame_to_color_optical_frame" type="fixed">
         <parent link="depth_camera_left_color_frame"/>
@@ -518,8 +443,5 @@
         <origin rpy="-1.57079632679 0.0 -1.57079632679" xyz="0.0 0.0 0.0"/>
     </joint>
-    <!-- Camera color optical link -->
     <link name="depth_camera_left_color_optical_frame"/>
-    <!-- Camera joint -->
-    <!-- Is located between the two back screw holes at ground level. -->
     <joint name="base_to_depth_camera_right_camera" type="fixed">
         <parent link="base"/>
@@ -527,5 +449,4 @@
         <origin rpy="0.0 0.523598775598 -1.57079632679" xyz="0.0 -0.07646 0.02905"/>
     </joint>
-    <!-- Camera link -->
     <link name="depth_camera_right_camera">
         <visual>
@@ -541,6 +462,4 @@
         </inertial>
     </link>
-    <!-- Camera parent joint -->
-    <!-- Frame lies on the left ir camera according to any_realsense2_camera urdf. -->
     <joint name="depth_camera_right_camera_to_camera_parent" type="fixed">
         <parent link="depth_camera_right_camera"/>
@@ -548,7 +467,5 @@
         <origin rpy="0.0 0.0 0.0" xyz="0.0255 0.0175 0.0"/>
     </joint>
-    <!-- Camera parent link -->
     <link name="depth_camera_right_camera_parent"/>
-    <!-- Depth optical frame joint -->
     <joint name="depth_camera_right_camera_parent_to_depth_optical_frame" type="fixed">
         <parent link="depth_camera_right_camera_parent"/>
@@ -556,7 +473,5 @@
         <origin rpy="-1.57079632679 0.0 -1.57079632679" xyz="0.0 0.0 0.0"/>
     </joint>
-    <!-- Depth optical frame link -->
     <link name="depth_camera_right_depth_optical_frame"/>
-    <!-- Camera color frame joint -->
     <joint name="depth_camera_right_camera_parent_to_color_frame" type="fixed">
         <parent link="depth_camera_right_camera_parent"/>
@@ -564,7 +479,5 @@
         <origin rpy="0 0 0" xyz="0 0.015 0"/>
     </joint>
-    <!-- Camera color frame link -->
     <link name="depth_camera_right_color_frame"/>
-    <!-- Camera color optical joint -->
     <joint name="depth_camera_right_color_frame_to_color_optical_frame" type="fixed">
         <parent link="depth_camera_right_color_frame"/>
@@ -572,7 +485,5 @@
         <origin rpy="-1.57079632679 0.0 -1.57079632679" xyz="0.0 0.0 0.0"/>
     </joint>
-    <!-- Camera color optical link -->
     <link name="depth_camera_right_color_optical_frame"/>
-    <!-- parent to cage joint, located between mounting plate on trunk and the cage -->
     <joint name="base_to_lidar_cage" type="fixed">
         <parent link="base"/>
@@ -580,5 +491,4 @@
         <origin rpy="0 0 0" xyz="-0.364 0.0 0.0735"/>
     </joint>
-    <!-- Velodyne cage link -->
     <link name="lidar_cage">
         <visual>
@@ -600,5 +510,4 @@
         </inertial>
     </link>
-    <!-- parent to sensor joint -->
     <joint name="lidar_cage_to_lidar" type="fixed">
         <parent link="lidar_cage"/>
@@ -606,5 +515,4 @@
         <origin rpy="0.0 0.0 -1.57079632679" xyz="0.0 0.0 0.0687"/>
     </joint>
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
File: urdf/anymal_gazebo.xacro (robot description, xacro)
@@ -12,5 +12,4 @@
         </joint>
     </xacro:macro>
-    <!-- ros2_control plugin -->
     <ros2_control name="GazeboSystem" type="system">
         <hardware>
@@ -42,5 +41,4 @@
         </sensor>
     </ros2_control>
-    <!-- Effort_controller -->
     <gazebo>
         <plugin filename="libgazebo_ros2_control.so" name="gazebo_ros2_control">
@@ -48,17 +46,8 @@
         </plugin>
     </gazebo>
-    <!-- IMU sensor -->
     <gazebo reference="base">
         <sensor name="imu_sensor" type="imu">
             <always_on>true</always_on>
             <update_rate>400</update_rate>
-            <!-- <plugin name="imu_plugin" filename="libgazebo_ros_imu_sensor.so">
-                <ros>
-                    <namespace>/imu</namespace>
-                    <remapping>~/out:=data</remapping>
-                </ros>
-                <frame_name>base</frame_name>
-                <initial_orientation_as_reference>true</initial_orientation_as_reference>
-            </plugin> -->
             <imu>
                 <angular_velocity>
@@ -117,6 +106,4 @@
         </sensor>
     </gazebo>
-    <!-- Contact sensors for the four feet -->
-    <!-- LF_FOOT -->
     <gazebo reference="LF_FOOT">
         <sensor name="LF_FOOT_contct_sensor" type="contact">
@@ -124,5 +111,4 @@
             <update_rate>25.0</update_rate>
             <contact>
-                <!-- gz sdf -p turtlebot3_burger.urdf.xacro and look for the name of the desired collision element. -->
                 <xacro:if value="${remove_shank_collisions}">
                     <collision>LF_SHANK_fixed_joint_lump__LF_FOOT_collision_2</collision>
@@ -134,5 +120,4 @@
             <plugin name="LF_FOOT_bumper" filename="libgazebo_ros_bumper.so">
                 <ros>
-                    <!-- <namespace>demo</namespace> -->
                     <remapping>bumper_states:=/contact_force_sensors/LF</remapping>
                 </ros>
@@ -141,5 +126,4 @@
         </sensor>
     </gazebo>
-    <!-- RF_FOOT -->
     <gazebo reference="RF_FOOT">
         <sensor name="RF_FOOT_contct_sensor" type="contact">
@@ -147,5 +131,4 @@
             <update_rate>25.0</update_rate>
             <contact>
-                <!-- gz sdf -p turtlebot3_burger.urdf.xacro and look for the name of the desired collision element. -->
                 <xacro:if value="${remove_shank_collisions}">
                     <collision>RF_SHANK_fixed_joint_lump__RF_FOOT_collision_2</collision>
@@ -157,5 +140,4 @@
             <plugin name="RF_FOOT_bumper" filename="libgazebo_ros_bumper.so">
                 <ros>
-                    <!-- <namespace>demo</namespace> -->
                     <remapping>bumper_states:=/contact_force_sensors/RF</remapping>
                 </ros>
@@ -164,5 +146,4 @@
         </sensor>
     </gazebo>
-    <!-- LH_FOOT -->
     <gazebo reference="LH_FOOT">
         <sensor name="LH_FOOT_contct_sensor" type="contact">
@@ -170,5 +151,4 @@
             <update_rate>25.0</update_rate>
             <contact>
-                <!-- gz sdf -p turtlebot3_burger.urdf.xacro and look for the name of the desired collision element. -->
                 <xacro:if value="${remove_shank_collisions}">
                     <collision>LH_SHANK_fixed_joint_lump__LH_FOOT_collision_2</collision>
@@ -180,5 +160,4 @@
             <plugin name="LH_FOOT_bumper" filename="libgazebo_ros_bumper.so">
                 <ros>
-                    <!-- <namespace>demo</namespace> -->
                     <remapping>bumper_states:=/contact_force_sensors/LH</remapping>
                 </ros>
@@ -187,5 +166,4 @@
         </sensor>
     </gazebo>
-    <!-- RH_FOOT -->
     <gazebo reference="RH_FOOT">
         <sensor name="RH_FOOT_contct_sensor" type="contact">
@@ -193,5 +171,4 @@
             <update_rate>25.0</update_rate>
             <contact>
-                <!-- gz sdf -p turtlebot3_burger.urdf.xacro and look for the name of the desired collision element. -->
                 <xacro:if value="${remove_shank_collisions}">
                     <collision>RH_SHANK_fixed_joint_lump__RH_FOOT_collision_2</collision>
@@ -203,5 +180,4 @@
             <plugin name="RH_FOOT_bumper" filename="libgazebo_ros_bumper.so">
                 <ros>
-                    <!-- <namespace>demo</namespace> -->
                     <remapping>bumper_states:=/contact_force_sensors/RH</remapping>
                 </ros>
