Commit message: Use package:// instead of file:// for meshes

File: urdf/anymal.urdf (robot description, URDF)
Before this commit: robot anymal, 78 links, 77 joints
Links:
- link LF_FOOT: geometry collision cylinder length=0.282504 radius=0.0175; collision sphere radius=0.03
- link LF_HAA: geometry visual mesh filename=package://anymal_c_simple_description/meshes/drive.dae scale=1.0 1.0 1.0
- link LF_HFE: geometry collision cylinder length=0.14 radius=0.05; visual mesh filename=package://anymal_c_simple_description/meshes/drive.dae scale=1.0 1.0 1.0
- link LF_KFE: geometry collision cylinder length=0.14 radius=0.05; visual mesh filename=package://anymal_c_simple_description/meshes/drive.dae scale=1.0 1.0 1.0
- link LF_hip_fixed: geometry visual mesh filename=package://anymal_c_simple_description/meshes/hip_l.dae scale=1.0 1.0 1.0
- link LF_shank_fixed: geometry collision box size=0.114998 0.0675 0.04; collision cylinder length=0.04 radius=0.06
- link LF_thigh_fixed: geometry collision box size=0.075 0.06 0.282627; collision cylinder length=0.08 radius=0.065
- link LH_FOOT: geometry collision cylinder length=0.282504 radius=0.0175; collision sphere radius=0.03
- link LH_HAA: geometry visual mesh filename=package://anymal_c_simple_description/meshes/drive.dae scale=1.0 1.0 1.0
- link LH_HFE: geometry collision cylinder length=0.14 radius=0.05; visual mesh filename=package://anymal_c_simple_description/meshes/drive.dae scale=1.0 1.0 1.0
- link LH_KFE: geometry collision cylinder length=0.14 radius=0.05; visual mesh filename=package://anymal_c_simple_description/meshes/drive.dae scale=1.0 1.0 1.0
- link LH_hip_fixed: geometry visual mesh filename=package://anymal_c_simple_description/meshes/hip_r.dae scale=1.0 1.0 1.0
- link LH_shank_fixed: geometry collision box size=0.114998 0.0675 0.04; collision cylinder length=0.04 radius=0.06
- link LH_thigh_fixed: geometry collision box size=0.075 0.06 0.282627; collision cylinder length=0.08 radius=0.065
- link RF_FOOT: geometry collision cylinder length=0.282504 radius=0.0175; collision sphere radius=0.03
- link RF_HAA: geometry visual mesh filename=package://anymal_c_simple_description/meshes/drive.dae scale=1.0 1.0 1.0
- link RF_HFE: geometry collision cylinder length=0.14 radius=0.05; visual mesh filename=package://anymal_c_simple_description/meshes/drive.dae scale=1.0 1.0 1.0
- link RF_KFE: geometry collision cylinder length=0.14 radius=0.05; visual mesh filename=package://anymal_c_simple_description/meshes/drive.dae scale=1.0 1.0 1.0
- link RF_hip_fixed: geometry visual mesh filename=package://anymal_c_simple_description/meshes/hip_r.dae scale=1.0 1.0 1.0
- link RF_shank_fixed: geometry collision box size=0.114998 0.0675 0.04; collision cylinder length=0.04 radius=0.06
- link RF_thigh_fixed: geometry collision box size=0.075 0.06 0.282627; collision cylinder length=0.08 radius=0.065
- link RH_FOOT: geometry collision cylinder length=0.282504 radius=0.0175; collision sphere radius=0.03
- link RH_HAA: geometry visual mesh filename=package://anymal_c_simple_description/meshes/drive.dae scale=1.0 1.0 1.0
- link RH_HFE: geometry collision cylinder length=0.14 radius=0.05; visual mesh filename=package://anymal_c_simple_description/meshes/drive.dae scale=1.0 1.0 1.0
- link RH_KFE: geometry collision cylinder length=0.14 radius=0.05; visual mesh filename=package://anymal_c_simple_description/meshes/drive.dae scale=1.0 1.0 1.0
- link RH_hip_fixed: geometry visual mesh filename=package://anymal_c_simple_description/meshes/hip_l.dae scale=1.0 1.0 1.0
- link RH_shank_fixed: geometry collision box size=0.114998 0.0675 0.04; collision cylinder length=0.04 radius=0.06
- link RH_thigh_fixed: geometry collision box size=0.075 0.06 0.282627; collision cylinder length=0.08 radius=0.065
- link base: geometry collision box size=0.58 0.14 0.18; collision cylinder length=0.145 radius=0.09
- link battery: geometry visual mesh filename=package://anymal_c_simple_description/meshes/battery.dae scale=1.0 1.0 1.0
- link bottom_shell: geometry visual mesh filename=package://anymal_c_simple_description/meshes/bottom_shell.d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 scale=1.0 1.0 1.0
- link depth_camera_front_camera: geometry visual mesh filename=package://anymal_c_simple_description/meshes/depth_camera.d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 scale=1.0 1.0 1.0
- link depth_camera_left_camera: geometry visual mesh filename=package://anymal_c_simple_description/meshes/depth_camera.d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 scale=1.0 1.0 1.0
- link depth_camera_rear_camera: geometry visual mesh filename=package://anymal_c_simple_description/meshes/depth_camera.d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 scale=1.0 1.0 1.0
- link depth_camera_right_camera: geometry visual mesh filename=package://anymal_c_simple_description/meshes/depth_camera.d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 scale=1.0 1.0 1.0
- link face_front: geometry collision box size=0.11 0.14 0.18; collision cylinder length=0.11 radius=0.09
- link face_rear: geometry collision box size=0.11 0.14 0.18; collision cylinder length=0.11 radius=0.09
- link handle: geometry visual mesh filename=package://anymal_c_simple_description/meshes/handle.dae scale=1.0 1.0 1.0
- link hatch: geometry visual mesh filename=package://anymal_c_simple_description/meshes/hatch.dae scale=1.0 1.0 1.0
- link lidar: geometry visual mesh filename=package://anymal_c_simple_description/meshes/lidar.dae
- link lidar_cage: geometry collision cylinder length=0.12 radius=0.07; visual mesh filename=package://anymal_c_simple_description/meshes/lidar_cage.dae scale=1.0 1.0 1.0
- link remote: geometry visual mesh filename=package://anymal_c_simple_description/meshes/remote.dae scale=1.0 1.0 1.0
- link top_shell: geometry visual mesh filename=package://anymal_c_simple_description/meshes/top_shell.dae scale=1.0 1.0 1.0
- link wide_angle_camera_front_camera: geometry visual mesh filename=package://anymal_c_simple_description/meshes/wide_angle_cam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 scale=1.0 1.0 1.0
- link wide_angle_camera_rear_camera: geometry visual mesh filename=package://anymal_c_simple_description/meshes/wide_angle_cam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 scale=1.0 1.0 1.0

File: urdf/anymal.xacro (robot description, xacro)
@@ -29,5 +29,5 @@
             <origin rpy="0 0 0" xyz="0 0 0"/>
             <geometry>
-                <mesh filename="file://$(find anymal_c_simple_description)/meshes/base.dae" scale="1.0 1.0 1.0"/>
+                <mesh filename="package://anymal_c_simple_description/meshes/base.dae" scale="1.0 1.0 1.0"/>
             </geometry>
         </visual>
@@ -95,5 +95,5 @@
             <origin rpy="0 0 0" xyz="0 0 0"/>
             <geometry>
-                <mesh filename="file://$(find anymal_c_simple_description)/meshes/top_shell.dae" scale="1.0 1.0 1.0"/>
+                <mesh filename="package://anymal_c_simple_description/meshes/top_shell.dae" scale="1.0 1.0 1.0"/>
             </geometry>
         </visual>
@@ -115,5 +115,5 @@
             <origin rpy="0 0 0" xyz="0 0 0"/>
             <geometry>
-                <mesh filename="file://$(find anymal_c_simple_description)/meshes/bottom_shell.dae" scale="1.0 1.0 1.0"/>
+                <mesh filename="package://anymal_c_simple_description/meshes/bottom_shell.dae" scale="1.0 1.0 1.0"/>
             </geometry>
         </visual>
@@ -135,5 +135,5 @@
             <origin rpy="0 0 0" xyz="0 0 0"/>
             <geometry>
-                <mesh filename="file://$(find anymal_c_simple_description)/meshes/remote.dae" scale="1.0 1.0 1.0"/>
+                <mesh filename="package://anymal_c_simple_description/meshes/remote.dae" scale="1.0 1.0 1.0"/>
             </geometry>
         </visual>
@@ -155,5 +155,5 @@
             <origin rpy="0 0 0" xyz="0 0 0"/>
             <geometry>
-                <mesh filename="file://$(find anymal_c_simple_description)/meshes/handle.dae" scale="1.0 1.0 1.0"/>
+                <mesh filename="package://anymal_c_simple_description/meshes/handle.dae" scale="1.0 1.0 1.0"/>
             </geometry>
         </visual>
@@ -175,5 +175,5 @@
             <origin rpy="0 0 0" xyz="0 0 0"/>
             <geometry>
-                <mesh filename="file://$(find anymal_c_simple_description)/meshes/face.dae" scale="1.0 1.0 1.0"/>
+                <mesh filename="package://anymal_c_simple_description/meshes/face.dae" scale="1.0 1.0 1.0"/>
             </geometry>
         </visual>
@@ -214,5 +214,5 @@
             <origin rpy="0 0 0" xyz="0.0 0.0 0.0"/>
             <geometry>
-                <mesh filename="file://$(find anymal_c_simple_description)/meshes/depth_camera.dae" scale="1.0 1.0 1.0"/>
+                <mesh filename="package://anymal_c_simple_description/meshes/depth_camera.dae" scale="1.0 1.0 1.0"/>
             </geometry>
         </visual>
@@ -268,5 +268,5 @@
             <origin rpy="0 0 0" xyz="0.0 0.0 0.0"/>
             <geometry>
-                <mesh filename="file://$(find anymal_c_simple_description)/meshes/wide_angle_camera.dae" scale="1.0 1.0 1.0"/>
+                <mesh filename="package://anymal_c_simple_description/meshes/wide_angle_camera.dae" scale="1.0 1.0 1.0"/>
             </geometry>
         </visual>
@@ -296,5 +296,5 @@
             <origin rpy="0 0 0" xyz="0 0 0"/>
             <geometry>
-                <mesh filename="file://$(find anymal_c_simple_description)/meshes/face.dae" scale="1.0 1.0 1.0"/>
+                <mesh filename="package://anymal_c_simple_description/meshes/face.dae" scale="1.0 1.0 1.0"/>
             </geometry>
         </visual>
@@ -335,5 +335,5 @@
             <origin rpy="0 0 0" xyz="0.0 0.0 0.0"/>
             <geometry>
-                <mesh filename="file://$(find anymal_c_simple_description)/meshes/depth_camera.dae" scale="1.0 1.0 1.0"/>
+                <mesh filename="package://anymal_c_simple_description/meshes/depth_camera.dae" scale="1.0 1.0 1.0"/>
             </geometry>
         </visual>
@@ -389,5 +389,5 @@
             <origin rpy="0 0 0" xyz="0.0 0.0 0.0"/>
             <geometry>
-                <mesh filename="file://$(find anymal_c_simple_description)/meshes/wide_angle_camera.dae" scale="1.0 1.0 1.0"/>
+                <mesh filename="package://anymal_c_simple_description/meshes/wide_angle_camera.dae" scale="1.0 1.0 1.0"/>
             </geometry>
         </visual>
@@ -417,5 +417,5 @@
             <origin rpy="0 0 0" xyz="0 0 0"/>
             <geometry>
-                <mesh filename="file://$(find anymal_c_simple_description)/meshes/battery.dae" scale="1.0 1.0 1.0"/>
+                <mesh filename="package://anymal_c_simple_description/meshes/battery.dae" scale="1.0 1.0 1.0"/>
             </geometry>
         </visual>
@@ -478,5 +478,5 @@
             <origin rpy="0 0 0" xyz="0.0 0.0 0.0"/>
             <geometry>
-                <mesh filename="file://$(find anymal_c_simple_description)/meshes/depth_camera.dae" scale="1.0 1.0 1.0"/>
+                <mesh filename="package://anymal_c_simple_description/meshes/depth_camera.dae" scale="1.0 1.0 1.0"/>
             </geometry>
         </visual>
@@ -532,5 +532,5 @@
             <origin rpy="0 0 0" xyz="0.0 0.0 0.0"/>
             <geometry>
-                <mesh filename="file://$(find anymal_c_simple_description)/meshes/depth_camera.dae" scale="1.0 1.0 1.0"/>
+                <mesh filename="package://anymal_c_simple_description/meshes/depth_camera.dae" scale="1.0 1.0 1.0"/>
             </geometry>
         </visual>
@@ -585,5 +585,5 @@
             <origin rpy="0.0 0.0 0.0" xyz="0.0 0.0 0.0"/>
             <geometry>
-                <mesh filename="file://$(find anymal_c_simple_description)/meshes/lidar_cage.dae" scale="1.0 1.0 1.0"/>
+                <mesh filename="package://anymal_c_simple_description/meshes/lidar_cage.dae" scale="1.0 1.0 1.0"/>
             </geometry>
         </visual>
@@ -616,5 +616,5 @@
             <origin xyz="0 0 0"/>
             <geometry>
-                <mesh filename="file://$(find anymal_c_simple_description)/meshes/lidar.dae"/>
+                <mesh filename="package://anymal_c_simple_description/meshes/lidar.dae"/>
             </geometry>
         </visual>
@@ -631,5 +631,5 @@
             <origin rpy="0 0 0" xyz="0 0 0"/>
             <geometry>
-                <mesh filename="file://$(find anymal_c_simple_description)/meshes/drive.dae" scale="1.0 1.0 1.0"/>
+                <mesh filename="package://anymal_c_simple_description/meshes/drive.dae" scale="1.0 1.0 1.0"/>
             </geometry>
         </visual>
@@ -668,5 +668,5 @@
             <origin rpy="0 0 0.0" xyz="0 0 0"/>
             <geometry>
-                <mesh filename="file://$(find anymal_c_simple_description)/meshes/hip_l.dae" scale="1.0 1.0 1.0"/>
+                <mesh filename="package://anymal_c_simple_description/meshes/hip_l.dae" scale="1.0 1.0 1.0"/>
             </geometry>
         </visual>
@@ -688,5 +688,5 @@
             <origin rpy="0 0 0" xyz="0 0 0"/>
             <geometry>
-                <mesh filename="file://$(find anymal_c_simple_description)/meshes/drive.dae" scale="1.0 1.0 1.0"/>
+                <mesh filename="package://anymal_c_simple_description/meshes/drive.dae" scale="1.0 1.0 1.0"/>
             </geometry>
         </visual>
@@ -731,5 +731,5 @@
             <origin rpy="0 0 0.0" xyz="0 0 0"/>
             <geometry>
-                <mesh filename="file://$(find anymal_c_simple_description)/meshes/thigh.dae" scale="1.0 1.0 1.0"/>
+                <mesh filename="package://anymal_c_simple_description/meshes/thigh.dae" scale="1.0 1.0 1.0"/>
             </geometry>
         </visual>
@@ -764,5 +764,5 @@
             <origin rpy="0 0 0" xyz="0 0 0"/>
             <geometry>
-                <mesh filename="file://$(find anymal_c_simple_description)/meshes/drive.dae" scale="1.0 1.0 1.0"/>
+                <mesh filename="package://anymal_c_simple_description/meshes/drive.dae" scale="1.0 1.0 1.0"/>
             </geometry>
         </visual>
@@ -807,5 +807,5 @@
             <origin rpy="0 0 0.0" xyz="0 0 0"/>
             <geometry>
-                <mesh filename="file://$(find anymal_c_simple_description)/meshes/shank_l.dae" scale="1.0 1.0 1.0"/>
+                <mesh filename="package://anymal_c_simple_description/meshes/shank_l.dae" scale="1.0 1.0 1.0"/>
             </geometry>
         </visual>
@@ -841,5 +841,5 @@
             <origin rpy="0 0 -0.785398163397" xyz="0 0 0"/>
             <geometry>
-                <mesh filename="file://$(find anymal_c_simple_description)/meshes/foot.dae" scale="1.0 1.0 1.0"/>
+                <mesh filename="package://anymal_c_simple_description/meshes/foot.dae" scale="1.0 1.0 1.0"/>
             </geometry>
         </visual>
@@ -877,5 +877,5 @@
             <origin rpy="0 0 0" xyz="0 0 0"/>
             <geometry>
-                <mesh filename="file://$(find anymal_c_simple_description)/meshes/drive.dae" scale="1.0 1.0 1.0"/>
+                <mesh filename="package://anymal_c_simple_description/meshes/drive.dae" scale="1.0 1.0 1.0"/>
             </geometry>
         </visual>
@@ -914,5 +914,5 @@
             <origin rpy="0 0 0.0" xyz="0 0 0"/>
             <geometry>
-                <mesh filename="file://$(find anymal_c_simple_description)/meshes/hip_r.dae" scale="1.0 1.0 1.0"/>
+                <mesh filename="package://anymal_c_simple_description/meshes/hip_r.dae" scale="1.0 1.0 1.0"/>
             </geometry>
         </visual>
@@ -934,5 +934,5 @@
             <origin rpy="0 0 0" xyz="0 0 0"/>
             <geometry>
-                <mesh filename="file://$(find anymal_c_simple_description)/meshes/drive.dae" scale="1.0 1.0 1.0"/>
+                <mesh filename="package://anymal_c_simple_description/meshes/drive.dae" scale="1.0 1.0 1.0"/>
             </geometry>
         </visual>
@@ -977,5 +977,5 @@
             <origin rpy="0 0 -3.14159265359" xyz="0 0 0"/>
             <geometry>
-                <mesh filename="file://$(find anymal_c_simple_description)/meshes/thigh.dae" scale="1.0 1.0 1.0"/>
+                <mesh filename="package://anymal_c_simple_description/meshes/thigh.dae" scale="1.0 1.0 1.0"/>
             </geometry>
         </visual>
@@ -1010,5 +1010,5 @@
             <origin rpy="0 0 0" xyz="0 0 0"/>
             <geometry>
-                <mesh filename="file://$(find anymal_c_simple_description)/meshes/drive.dae" scale="1.0 1.0 1.0"/>
+                <mesh filename="package://anymal_c_simple_description/meshes/drive.dae" scale="1.0 1.0 1.0"/>
             </geometry>
         </visual>
@@ -1053,5 +1053,5 @@
             <origin rpy="0 0 0.0" xyz="0 0 0"/>
             <geometry>
-                <mesh filename="file://$(find anymal_c_simple_description)/meshes/shank_r.dae" scale="1.0 1.0 1.0"/>
+                <mesh filename="package://anymal_c_simple_description/meshes/shank_r.dae" scale="1.0 1.0 1.0"/>
             </geometry>
         </visual>
@@ -1087,5 +1087,5 @@
             <origin rpy="0 0 0.785398163397" xyz="0 0 0"/>
             <geometry>
-                <mesh filename="file://$(find anymal_c_simple_description)/meshes/foot.dae" scale="1.0 1.0 1.0"/>
+                <mesh filename="package://anymal_c_simple_description/meshes/foot.dae" scale="1.0 1.0 1.0"/>
             </geometry>
         </visual>
@@ -1123,5 +1123,5 @@
             <origin rpy="0 0 0" xyz="0 0 0"/>
             <geometry>
-                <mesh filename="file://$(find anymal_c_simple_description)/meshes/drive.dae" scale="1.0 1.0 1.0"/>
+                <mesh filename="package://anymal_c_simple_description/meshes/drive.dae" scale="1.0 1.0 1.0"/>
             </geometry>
         </visual>
@@ -1160,5 +1160,5 @@
             <origin rpy="0 0 -3.14159265359" xyz="0 0 0"/>
             <geometry>
-                <mesh filename="file://$(find anymal_c_simple_description)/meshes/hip_r.dae" scale="1.0 1.0 1.0"/>
+                <mesh filename="package://anymal_c_simple_description/meshes/hip_r.dae" scale="1.0 1.0 1.0"/>
             </geometry>
         </visual>
@@ -1180,5 +1180,5 @@
             <origin rpy="0 0 0" xyz="0 0 0"/>
             <geometry>
-                <mesh filename="file://$(find anymal_c_simple_description)/meshes/drive.dae" scale="1.0 1.0 1.0"/>
+                <mesh filename="package://anymal_c_simple_description/meshes/drive.dae" scale="1.0 1.0 1.0"/>
             </geometry>
         </visual>
@@ -1223,5 +1223,5 @@
             <origin rpy="0 0 0.0" xyz="0 0 0"/>
             <geometry>
-                <mesh filename="file://$(find anymal_c_simple_description)/meshes/thigh.dae" scale="1.0 1.0 1.0"/>
+                <mesh filename="package://anymal_c_simple_description/meshes/thigh.dae" scale="1.0 1.0 1.0"/>
             </geometry>
         </visual>
@@ -1256,5 +1256,5 @@
             <origin rpy="0 0 0" xyz="0 0 0"/>
             <geometry>
-                <mesh filename="file://$(find anymal_c_simple_description)/meshes/drive.dae" scale="1.0 1.0 1.0"/>
+                <mesh filename="package://anymal_c_simple_description/meshes/drive.dae" scale="1.0 1.0 1.0"/>
             </geometry>
         </visual>
@@ -1299,5 +1299,5 @@
             <origin rpy="0 0 -3.14159265359" xyz="0 0 0"/>
             <geometry>
-                <mesh filename="file://$(find anymal_c_simple_description)/meshes/shank_r.dae" scale="1.0 1.0 1.0"/>
+                <mesh filename="package://anymal_c_simple_description/meshes/shank_r.dae" scale="1.0 1.0 1.0"/>
             </geometry>
         </visual>
@@ -1333,5 +1333,5 @@
             <origin rpy="0 0 -2.35619449019" xyz="0 0 0"/>
             <geometry>
-                <mesh filename="file://$(find anymal_c_simple_description)/meshes/foot.dae" scale="1.0 1.0 1.0"/>
+                <mesh filename="package://anymal_c_simple_description/meshes/foot.dae" scale="1.0 1.0 1.0"/>
             </geometry>
         </visual>
@@ -1369,5 +1369,5 @@
             <origin rpy="0 0 0" xyz="0 0 0"/>
             <geometry>
-                <mesh filename="file://$(find anymal_c_simple_description)/meshes/drive.dae" scale="1.0 1.0 1.0"/>
+                <mesh filename="package://anymal_c_simple_description/meshes/drive.dae" scale="1.0 1.0 1.0"/>
             </geometry>
         </visual>
@@ -1406,5 +1406,5 @@
             <origin rpy="0 0 -3.14159265359" xyz="0 0 0"/>
             <geometry>
-                <mesh filename="file://$(find anymal_c_simple_description)/meshes/hip_l.dae" scale="1.0 1.0 1.0"/>
+                <mesh filename="package://anymal_c_simple_description/meshes/hip_l.dae" scale="1.0 1.0 1.0"/>
             </geometry>
         </visual>
@@ -1426,5 +1426,5 @@
             <origin rpy="0 0 0" xyz="0 0 0"/>
             <geometry>
-                <mesh filename="file://$(find anymal_c_simple_description)/meshes/drive.dae" scale="1.0 1.0 1.0"/>
+                <mesh filename="package://anymal_c_simple_description/meshes/drive.dae" scale="1.0 1.0 1.0"/>
             </geometry>
         </visual>
@@ -1469,5 +1469,5 @@
             <origin rpy="0 0 -3.14159265359" xyz="0 0 0"/>
             <geometry>
-                <mesh filename="file://$(find anymal_c_simple_description)/meshes/thigh.dae" scale="1.0 1.0 1.0"/>
+                <mesh filename="package://anymal_c_simple_description/meshes/thigh.dae" scale="1.0 1.0 1.0"/>
             </geometry>
         </visual>
@@ -1502,5 +1502,5 @@
             <origin rpy="0 0 0" xyz="0 0 0"/>
             <geometry>
-                <mesh filename="file://$(find anymal_c_simple_description)/meshes/drive.dae" scale="1.0 1.0 1.0"/>
+                <mesh filename="package://anymal_c_simple_description/meshes/drive.dae" scale="1.0 1.0 1.0"/>
             </geometry>
         </visual>
@@ -1545,5 +1545,5 @@
             <origin rpy="0 0 -3.14159265359" xyz="0 0 0"/>
             <geometry>
-                <mesh filename="file://$(find anymal_c_simple_description)/meshes/shank_l.dae" scale="1.0 1.0 1.0"/>
+                <mesh filename="package://anymal_c_simple_description/meshes/shank_l.dae" scale="1.0 1.0 1.0"/>
             </geometry>
         </visual>
@@ -1579,5 +1579,5 @@
             <origin rpy="0 0 -3.92699081699" xyz="0 0 0"/>
             <geometry>
-                <mesh filename="file://$(find anymal_c_simple_description)/meshes/foot.dae" scale="1.0 1.0 1.0"/>
+                <mesh filename="package://anymal_c_simple_description/meshes/foot.dae" scale="1.0 1.0 1.0"/>
             </geometry>
         </visual>
@@ -1615,5 +1615,5 @@
             <origin rpy="0 0 0" xyz="0.116 0 0.073"/>
             <geometry>
-                <mesh filename="file://$(find anymal_c_simple_description)/meshes/hatch.dae" scale="1.0 1.0 1.0"/>
+                <mesh filename="package://anymal_c_simple_description/meshes/hatch.dae" scale="1.0 1.0 1.0"/>
             </geometry>
         </visual>
